Commit message: 3D stack: skid-steer friction, progress checker tolerance, re-route after failed segments, motion diagnostics
Co-Authored-By: Claude Opus 5.5 <noreply@anthropic.com>
Claude-Session: https://claude.ai/code/session_013ipojUcp5zwTno7wEzBHPa

File: ros2_ws/src/trecsar_description/urdf/trecsar.urdf.xacro (robot description, xacro)
@@ -54,5 +54,5 @@
     </joint>
     <gazebo reference="${name}">
-      <collision><surface><friction><ode><mu>1.2</mu><mu2>0.6</mu2></ode></friction></surface></collision>
+      <collision><surface><friction><ode><mu>1.0</mu><mu2>0.25</mu2></ode></friction></surface></collision>
     </gazebo>
   </xacro:macro>

Commit message: UGV model: traction on centre wheels, low-friction end wheels so the tracked robot can pivot
Diagnostics showed Nav2 commanding in-place rotation that the 6-wheel skid model
could not execute.

Co-Authored-By: Claude Opus 5.5 <noreply@anthropic.com>
Claude-Session: https://claude.ai/code/session_013ipojUcp5zwTno7wEzBHPa

File: ros2_ws/src/trecsar_description/urdf/trecsar.urdf.xacro (robot description, xacro)
@@ -44,6 +44,8 @@
   <xacro:track_belt side="left" y="${track_y}"/>
   <xacro:track_belt side="right" y="${-track_y}"/>
-  <!-- road wheels (physics) -->
-  <xacro:macro name="wheel" params="name x y">
+  <!-- road wheels (physics). Tracks are approximated the usual way for Gazebo: the centre
+       wheels carry the traction and the front/rear wheels are low-friction, so the robot can
+       pivot on the spot like the real tracked platform instead of jamming in a 6-wheel skid. -->
+  <xacro:macro name="wheel" params="name x y mu">
     <link name="${name}">
       <collision><origin rpy="${pi/2} 0 0"/><geometry><cylinder radius="${wheel_r}" length="${wheel_w}"/></geometry></collision>
@@ -54,13 +56,13 @@
     </joint>
     <gazebo reference="${name}">
-      <collision><surface><friction><ode><mu>1.0</mu><mu2>0.25</mu2></ode></friction></surface></collision>
+      <mu1>${mu}</mu1><mu2>${mu}</mu2>  <!-- sdformat converts these into the collision surface -->
     </gazebo>
   </xacro:macro>
-  <xacro:wheel name="left_front" x="${L/2 - wheel_r}" y="${track_y}"/>
-  <xacro:wheel name="left_mid" x="0" y="${track_y}"/>
-  <xacro:wheel name="left_rear" x="${-L/2 + wheel_r}" y="${track_y}"/>
-  <xacro:wheel name="right_front" x="${L/2 - wheel_r}" y="${-track_y}"/>
-  <xacro:wheel name="right_mid" x="0" y="${-track_y}"/>
-  <xacro:wheel name="right_rear" x="${-L/2 + wheel_r}" y="${-track_y}"/>
+  <xacro:wheel name="left_front" x="${L/2 - wheel_r}" y="${track_y}" mu="0.05"/>
+  <xacro:wheel name="left_mid" x="0" y="${track_y}" mu="1.0"/>
+  <xacro:wheel name="left_rear" x="${-L/2 + wheel_r}" y="${track_y}" mu="0.05"/>
+  <xacro:wheel name="right_front" x="${L/2 - wheel_r}" y="${-track_y}" mu="0.05"/>
+  <xacro:wheel name="right_mid" x="0" y="${-track_y}" mu="1.0"/>
+  <xacro:wheel name="right_rear" x="${-L/2 + wheel_r}" y="${-track_y}" mu="0.05"/>
   <!-- sensor mast: RGB camera + thermal camera -->
   <link name="mast">

Commit message: Mount the lidar on top of the mast: it was seeing the robot's own relay bay
Nav2's controller aborted with 'collision ahead' because the scan plane crossed
the relay bay. Regression test checks that no robot part crosses the scan plane.

Co-Authored-By: Claude Opus 5.5 <noreply@anthropic.com>
Claude-Session: https://claude.ai/code/session_013ipojUcp5zwTno7wEzBHPa

File: ros2_ws/src/trecsar_description/urdf/trecsar.urdf.xacro (robot description, xacro)
@@ -82,9 +82,11 @@
   </link>
   <joint name="thermal_joint" type="fixed"><parent link="mast"/><child link="thermal_link"/><origin xyz="0.03 0 0.44"/></joint>
-  <!-- 3D lidar for SLAM / Nav2 -->
+  <!-- 2D lidar for SLAM / Nav2 -->
   <link name="lidar_link">
     <visual><geometry><cylinder radius="0.05" length="0.07"/></geometry><material name="black"/></visual>
   </link>
-  <joint name="lidar_joint" type="fixed"><parent link="base_link"/><child link="lidar_link"/><origin xyz="0.05 0 ${H + 0.05}"/></joint>
+  <!-- on top of the mast, above every part of the robot: a lower mount let the lidar see the
+       relay bay, which Nav2 then treated as a permanent obstacle -->
+  <joint name="lidar_joint" type="fixed"><parent link="mast"/><child link="lidar_link"/><origin xyz="0 0 0.62"/></joint>
   <link name="imu_link"/>
   <joint name="imu_joint" type="fixed"><parent link="base_link"/><child link="imu_link"/><origin xyz="0 0 0.05"/></joint>
